Commit message: 20250814

File: install/workcell_description/share/workcell_description/urdf/props/common_props.xacro (robot description, xacro)
@@ -1,2 +1,3 @@
+<!--
 <?xml version="1.0"?>
 <robot xmlns:xacro="http://ros.org/wiki/xacro">
@@ -11,2 +12,16 @@
   <xacro:property name="d415_rpy"  value="0 0 0"/>
 </robot>
+-->
+<?xml version="1.0"?>
+<robot xmlns:xacro="http://ros.org/wiki/xacro">
+  <!-- 可覆盖参数（默认值） -->
+  <xacro:arg name="prefix"                default=""/>
+  <xacro:arg name="mesh_scale_visual"     default="1 1 1"/>
+  <xacro:arg name="mesh_scale_collision"  default="1 1 1"/>
+  <!-- 转成全局属性 -->
+  <xacro:property name="prefix"               value="$(arg prefix)"/>
+  <xacro:property name="mesh_scale_visual"    value="$(arg mesh_scale_visual)"/>
+  <xacro:property name="mesh_scale_collision" value="$(arg mesh_scale_collision)"/>
+  <!-- 小工具：角度→弧度 -->
+  <xacro:property name="deg" value="0.017453292519943295"/>
+</robot>

File: install/workcell_description/share/workcell_description/urdf/robots/irb6700_200_260.xacro (robot description, xacro)
@@ -3,5 +3,6 @@
   <!-- include common materials -->
   <xacro:include filename="../materials/common_materials.xacro"/>
-  <xacro:macro name="irb6700_200_260" params="prefix">
+<xacro:macro name="irb6700_200_260"
+             params="prefix mesh_scale_visual:='1 1 1' mesh_scale_collision:='1 1 1'">
     <!-- === link list === -->
     <link name="${prefix}base_link">

File: install/workcell_description/share/workcell_description/urdf/workcell.urdf.xacro (robot description, xacro)
@@ -5,4 +5,5 @@
   <xacro:include filename="materials/common_materials.xacro"/>
   <xacro:include filename="robots/irb6700_200_260.xacro"/>
+  <xacro:include filename="actuators/spindle.xacro"/>
   <!-- 机器人主体 -->
   <xacro:irb6700_200_260 prefix="${prefix}"
@@ -12,7 +13,10 @@
   <xacro:irb6700_tcp_frames prefix="${prefix}"/>
   <!-- 末端执行器 -->
-  <xacro:mount_ee_tool prefix="${prefix}" parent_link="tool0" xyz="0 0 0" rpy="0 0 0"
-      scale_v="${mesh_scale_visual}" scale_c="${mesh_scale_collision}"/>
-  <!-- 手眼/固定相机（带开关） -->
+  <xacro:mount_spindle prefix="${prefix}"
+    parent_link:="tool0"
+    mount_xyz:="0 0 0" mount_rpy:="0 0 0"
+    scale_v:="${mesh_scale_visual}" scale_c:="${mesh_scale_collision}"
+    tcp_offset:="0.150"/>
+  <!-- 手眼/固定相机（带开关）
   <xacro:if value="${use_d435i}">
     <xacro:mount_d435i prefix="${prefix}" parent_link="tool0"
@@ -24,5 +28,6 @@
         xyz="${d415_xyz}" rpy="${d415_rpy}"/>
   </xacro:if>
-  <!-- 场地 -->
+  场地
   <xacro:add_table prefix="${prefix}" base="base_link" xyz="0.8 0 0" rpy="0 0 0"/>
+  -->
 </robot>

File: src/workcell_description/urdf/workcell.urdf.xacro (robot description, xacro)
@@ -18,5 +18,5 @@
     scale_v:="${mesh_scale_visual}" scale_c:="${mesh_scale_collision}"
     tcp_offset:="0.150"/>
-  <!-- 手眼/固定相机（带开关） -->
+  <!-- 手眼/固定相机（带开关）
   <xacro:if value="${use_d435i}">
     <xacro:mount_d435i prefix="${prefix}" parent_link="tool0"
@@ -28,5 +28,6 @@
         xyz="${d415_xyz}" rpy="${d415_rpy}"/>
   </xacro:if>
-  <!-- 场地 -->
+  场地
   <xacro:add_table prefix="${prefix}" base="base_link" xyz="0.8 0 0" rpy="0 0 0"/>
+  -->
 </robot>
