Commit message: heng

File: install/workcell_description/share/workcell_description/urdf/actuators/spindle.xacro (robot description, xacro)
@@ -7,5 +7,5 @@
                        mount_xyz:='0 0 0' mount_rpy:='0 0 0'
                        scale_v:='1 1 1' scale_c:='1 1 1'
-                       tcp_offset:='0.2595'   <!-- 150mm，按实物改 -->
+                       tcp_offset:='0.2595'
                        mass:='3.0'
                        ixx:='0.01' iyy:='0.01' izz:='0.005'">

File: install/workcell_description/share/workcell_description/urdf/props/common_props.xacro (robot description, xacro)
@@ -1,16 +1,2 @@
-<!--
-<?xml version="1.0"?>
-<robot xmlns:xacro="http://ros.org/wiki/xacro">
-  <xacro:property name="prefix"                value=""/>
-  <xacro:property name="mesh_scale_visual"     value="1 1 1"/>
-  <xacro:property name="mesh_scale_collision"  value="1 1 1"/>
-  <xacro:property name="use_d435i" value="true"/>
-  <xacro:property name="use_d415"  value="true"/>
-  <xacro:property name="d435i_xyz" value="0.08 0.00 0.02"/>
-  <xacro:property name="d435i_rpy" value="0 0 1.5708"/>
-  <xacro:property name="d415_xyz"  value="0.80 0.00 1.20"/>
-  <xacro:property name="d415_rpy"  value="0 0 0"/>
-</robot>
--->
 <?xml version="1.0"?>
 <robot xmlns:xacro="http://ros.org/wiki/xacro">

File: install/workcell_description/share/workcell_description/urdf/workcell.urdf.xacro (robot description, xacro)
@@ -1,18 +1,17 @@
 <?xml version="1.0" encoding="UTF-8"?>
-<robot xmlns:xacro="http://ros.org/wiki/xacro" name="workcell">
-  <!-- 全局参数与材质 -->
+<robot xmlns:xacro="http://www.ros.org/wiki/xacro" name="workcell">
   <xacro:include filename="props/common_props.xacro"/>
   <xacro:include filename="materials/common_materials.xacro"/>
   <xacro:include filename="robots/irb6700_200_260.xacro"/>
   <xacro:include filename="actuators/spindle.xacro"/>
-  <!-- 机器人主体 -->
-  <xacro:irb6700_200_260 prefix="${prefix}"
+  <xacro:irb6700_200_260
+      prefix="${prefix}"
       mesh_scale_visual="${mesh_scale_visual}"
       mesh_scale_collision="${mesh_scale_collision}"/>
-  <!-- 末端执行器 -->
-  <xacro:mount_spindle prefix="${prefix}"
-    parent_link:="${prefix}tool0"
-    mount_xyz:="0 0 0" mount_rpy:="0 0 0"
-    scale_v:="${mesh_scale_visual}" scale_c:="${mesh_scale_collision}"
-    tcp_offset:="0.150"/>
+  <xacro:mount_spindle
+      prefix="${prefix}"
+      parent_link="tool0"
+      mount_xyz="0 0 0" mount_rpy="0 0 0"
+      scale_v="${mesh_scale_visual}" scale_c="${mesh_scale_collision}"
+      tcp_offset="0.150"/>
 </robot>
