Commit message: heng

File: install/workcell_description/share/workcell_description/urdf/materials/common_materials.xacro (robot description, xacro)
@@ -2,78 +2,95 @@
 <robot xmlns:xacro="http://ros.org/wiki/xacro">
   <xacro:include filename="../materials/common_colours.xacro"/>
+  <!-- Global material definitions for reuse across links -->
+  <material name="abb_orange">
+    <color rgba="${colour_abb_orange}"/>
+  </material>
+  <material name="abb_graphite_white">
+    <color rgba="${colour_abb_graphite_white}"/>
+  </material>
+  <material name="abb_white">
+    <color rgba="${colour_abb_white}"/>
+  </material>
+  <material name="abb_pebble_gray">
+    <color rgba="${colour_abb_pebble_gray}"/>
+  </material>
+  <material name="abb_dark_gray">
+    <color rgba="${colour_abb_dark_gray}"/>
+  </material>
+  <material name="abb_black">
+    <color rgba="${colour_abb_black}"/>
+  </material>
+  <material name="abb_signal_red">
+    <color rgba="${colour_abb_signal_red}"/>
+  </material>
+  <material name="abb_carmine_red">
+    <color rgba="${colour_abb_carmine_red}"/>
+  </material>
+  <material name="abb_ultramarine_blue">
+    <color rgba="${colour_abb_ultramarine_blue}"/>
+  </material>
+  <material name="abb_sky_blue">
+    <color rgba="${colour_abb_sky_blue}"/>
+  </material>
+  <material name="abb_leaf_green">
+    <color rgba="${colour_abb_leaf_green}"/>
+  </material>
+  <material name="abb_olive_green">
+    <color rgba="${colour_abb_olive_green}"/>
+  </material>
+  <material name="abb_gray_white">
+    <color rgba="${colour_abb_gray_white}"/>
+  </material>
+  <material name="abb_pure_white">
+    <color rgba="${colour_abb_pure_white}"/>
+  </material>
+  <material name="abb_yellow">
+    <color rgba="${colour_abb_yellow}"/>
+  </material>
+  <!-- Convenience macros referencing the named materials -->
   <xacro:macro name="material_abb_orange">
-    <material name="">
-      <color rgba="${colour_abb_orange}"/>
-    </material>
+    <material name="abb_orange"/>
   </xacro:macro>
   <xacro:macro name="material_abb_graphite_white">
-    <material name="">
-      <color rgba="${colour_abb_graphite_white}"/>
-    </material>
+    <material name="abb_graphite_white"/>
   </xacro:macro>
   <xacro:macro name="material_abb_white">
-    <material name="">
-      <color rgba="${colour_abb_white}"/>
-    </material>
+    <material name="abb_white"/>
   </xacro:macro>
   <xacro:macro name="material_abb_pebble_gray">
-    <material name="">
-      <color rgba="${colour_abb_pebble_gray}"/>
-    </material>
+    <material name="abb_pebble_gray"/>
   </xacro:macro>
   <xacro:macro name="material_abb_dark_gray">
-    <material name="">
-      <color rgba="${colour_abb_dark_gray}"/>
-    </material>
+    <material name="abb_dark_gray"/>
   </xacro:macro>
   <xacro:macro name="material_abb_black">
-    <material name="">
-      <color rgba="${colour_abb_black}"/>
-    </material>
+    <material name="abb_black"/>
   </xacro:macro>
   <xacro:macro name="material_abb_signal_red">
-    <material name="">
-      <color rgba="${colour_abb_signal_red}"/>
-    </material>
+    <material name="abb_signal_red"/>
   </xacro:macro>
   <xacro:macro name="material_abb_carmine_red">
-    <material name="">
-      <color rgba="${colour_abb_carmine_red}"/>
-    </material>
+    <material name="abb_carmine_red"/>
   </xacro:macro>
   <xacro:macro name="material_abb_ultramarine_blue">
-    <material name="">
-      <color rgba="${colour_abb_ultramarine_blue}"/>
-    </material>
+    <material name="abb_ultramarine_blue"/>
   </xacro:macro>
   <xacro:macro name="material_abb_sky_blue">
-    <material name="">
-      <color rgba="${colour_abb_sky_blue}"/>
-    </material>
+    <material name="abb_sky_blue"/>
   </xacro:macro>
   <xacro:macro name="material_abb_leaf_green">
-    <material name="">
-      <color rgba="${colour_abb_leaf_green}"/>
-    </material>
+    <material name="abb_leaf_green"/>
   </xacro:macro>
   <xacro:macro name="material_abb_olive_green">
-    <material name="">
-      <color rgba="${colour_abb_olive_green}"/>
-    </material>
+    <material name="abb_olive_green"/>
   </xacro:macro>
   <xacro:macro name="material_abb_gray_white">
-    <material name="">
-      <color rgba="${colour_abb_gray_white}"/>
-    </material>
+    <material name="abb_gray_white"/>
   </xacro:macro>
   <xacro:macro name="material_abb_pure_white">
-    <material name="">
-      <color rgba="${colour_abb_pure_white}"/>
-    </material>
+    <material name="abb_pure_white"/>
   </xacro:macro>
   <xacro:macro name="material_abb_yellow">
-    <material name="">
-      <color rgba="${colour_abb_yellow}"/>
-    </material>
+    <material name="abb_yellow"/>
   </xacro:macro>
 </robot>

File: install/workcell_description/share/workcell_description/urdf/robots/irb6700_200_260.xacro (robot description, xacro)
@@ -50,36 +50,13 @@
       </collision>
     </link>
-    <!-- Each link below now contains inertial placeholders -->
-    <xacro:macro name="irb6700_link" params="name mass ixx iyy izz">
-      <link name="${prefix}${name}">
-        <inertial>
-          <mass value="${mass}"/>
-          <origin xyz="0 0 0.1"/>
-          <inertia ixx="${ixx}" ixy="0" ixz="0" iyy="${iyy}" iyz="0" izz="${izz}"/>
-        </inertial>
-        <visual>
-          <origin xyz="0 0 0" rpy="0 0 0"/>
-          <geometry>
-            <mesh filename="package://workcell_description/meshes/robots/visual/${name}.stl" scale="${mesh_scale_visual}"/>
-          </geometry>
-          <xacro:material_abb_white/>
-        </visual>
-        <collision>
-          <origin xyz="0 0 0" rpy="0 0 0"/>
-          <geometry>
-            <mesh filename="package://workcell_description/meshes/robots/collision/${name}.stl" scale="${mesh_scale_collision}"/>
-          </geometry>
-          <xacro:material_abb_yellow/>
-        </collision>
-      </link>
-    </xacro:macro>
-    <xacro:irb6700_link name="link_1" mass="30.0" ixx="0.5" iyy="0.5" izz="0.5"/>
-    <xacro:irb6700_link name="link_2" mass="35.0" ixx="0.6" iyy="0.6" izz="0.6"/>
-    <xacro:irb6700_link name="link_3" mass="25.0" ixx="0.4" iyy="0.4" izz="0.4"/>
-    <xacro:irb6700_link name="link_4" mass="20.0" ixx="0.3" iyy="0.3" izz="0.3"/>
-    <xacro:irb6700_link name="link_5" mass="15.0" ixx="0.2" iyy="0.2" izz="0.2"/>
-    <xacro:irb6700_link name="link_6" mass="10.0" ixx="0.1" iyy="0.1" izz="0.1"/>
-    <xacro:irb6700_link name="cylinder" mass="5.0" ixx="0.05" iyy="0.05" izz="0.05"/>
-    <xacro:irb6700_link name="piston" mass="3.0" ixx="0.03" iyy="0.03" izz="0.03"/>
+    <!-- Each link below now uses the shared irb6700_link macro -->
+    <xacro:irb6700_link prefix="${prefix}" mesh_scale_visual="${mesh_scale_visual}" mesh_scale_collision="${mesh_scale_collision}" name="link_1" mass="30.0" ixx="0.5" iyy="0.5" izz="0.5"/>
+    <xacro:irb6700_link prefix="${prefix}" mesh_scale_visual="${mesh_scale_visual}" mesh_scale_collision="${mesh_scale_collision}" name="link_2" mass="35.0" ixx="0.6" iyy="0.6" izz="0.6"/>
+    <xacro:irb6700_link prefix="${prefix}" mesh_scale_visual="${mesh_scale_visual}" mesh_scale_collision="${mesh_scale_collision}" name="link_3" mass="25.0" ixx="0.4" iyy="0.4" izz="0.4"/>
+    <xacro:irb6700_link prefix="${prefix}" mesh_scale_visual="${mesh_scale_visual}" mesh_scale_collision="${mesh_scale_collision}" name="link_4" mass="20.0" ixx="0.3" iyy="0.3" izz="0.3"/>
+    <xacro:irb6700_link prefix="${prefix}" mesh_scale_visual="${mesh_scale_visual}" mesh_scale_collision="${mesh_scale_collision}" name="link_5" mass="15.0" ixx="0.2" iyy="0.2" izz="0.2"/>
+    <xacro:irb6700_link prefix="${prefix}" mesh_scale_visual="${mesh_scale_visual}" mesh_scale_collision="${mesh_scale_collision}" name="link_6" mass="10.0" ixx="0.1" iyy="0.1" izz="0.1"/>
+    <xacro:irb6700_link prefix="${prefix}" mesh_scale_visual="${mesh_scale_visual}" mesh_scale_collision="${mesh_scale_collision}" name="cylinder" mass="5.0" ixx="0.05" iyy="0.05" izz="0.05"/>
+    <xacro:irb6700_link prefix="${prefix}" mesh_scale_visual="${mesh_scale_visual}" mesh_scale_collision="${mesh_scale_collision}" name="piston" mass="3.0" ixx="0.03" iyy="0.03" izz="0.03"/>
     <!-- Add dynamics to joints -->
     <xacro:macro name="joint_dynamics" params="damping friction">
@@ -143,4 +120,13 @@
       <limit lower="-0.284" upper="0.371" effort="100" velocity="1.0"/>
     </joint>
+    <!-- Virtual prismatic joint to provide displacement equivalent to joint_2 rotation -->
+    <link name="${prefix}joint_2_slider"/>
+    <joint name="${prefix}joint_2_slider_joint" type="prismatic">
+      <origin xyz="0 0 0" rpy="0 0 0" />
+      <parent link="${prefix}link_1" />
+      <child link="${prefix}joint_2_slider" />
+      <axis xyz="0 1 0" />
+      <limit lower="-0.25" upper="0.25" effort="100" velocity="1.0" />
+    </joint>
     <joint name="${prefix}piston_joint" type="prismatic">
       <origin xyz="0 0 0" rpy="0.20897 0 -1.5708" />
@@ -148,5 +134,5 @@
       <child link="${prefix}piston" />
       <axis xyz="0 1 0" />
-      <mimic joint="${prefix}joint_2" multiplier="0.15"/>
+      <mimic joint="${prefix}joint_2_slider_joint" multiplier="1.0"/>
       <limit lower="-0.25" upper="0.25" effort="100" velocity="1.0" />
     </joint>

File: src/workcell_description/urdf/materials/common_materials.xacro (robot description, xacro)
@@ -2,78 +2,48 @@
 <robot xmlns:xacro="http://ros.org/wiki/xacro">
   <xacro:include filename="../materials/common_colours.xacro"/>
-  <xacro:macro name="material_abb_orange">
-    <material name="">
-      <color rgba="${colour_abb_orange}"/>
-    </material>
-  </xacro:macro>
-  <xacro:macro name="material_abb_graphite_white">
-    <material name="">
-      <color rgba="${colour_abb_graphite_white}"/>
-    </material>
-  </xacro:macro>
-  <xacro:macro name="material_abb_white">
-    <material name="">
-      <color rgba="${colour_abb_white}"/>
-    </material>
-  </xacro:macro>
-  <xacro:macro name="material_abb_pebble_gray">
-    <material name="">
-      <color rgba="${colour_abb_pebble_gray}"/>
-    </material>
-  </xacro:macro>
-  <xacro:macro name="material_abb_dark_gray">
-    <material name="">
-      <color rgba="${colour_abb_dark_gray}"/>
-    </material>
-  </xacro:macro>
-  <xacro:macro name="material_abb_black">
-    <material name="">
-      <color rgba="${colour_abb_black}"/>
-    </material>
-  </xacro:macro>
-  <xacro:macro name="material_abb_signal_red">
-    <material name="">
-      <color rgba="${colour_abb_signal_red}"/>
-    </material>
-  </xacro:macro>
-  <xacro:macro name="material_abb_carmine_red">
-    <material name="">
-      <color rgba="${colour_abb_carmine_red}"/>
-    </material>
-  </xacro:macro>
-  <xacro:macro name="material_abb_ultramarine_blue">
-    <material name="">
-      <color rgba="${colour_abb_ultramarine_blue}"/>
-    </material>
-  </xacro:macro>
-  <xacro:macro name="material_abb_sky_blue">
-    <material name="">
-      <color rgba="${colour_abb_sky_blue}"/>
-    </material>
-  </xacro:macro>
-  <xacro:macro name="material_abb_leaf_green">
-    <material name="">
-      <color rgba="${colour_abb_leaf_green}"/>
-    </material>
-  </xacro:macro>
-  <xacro:macro name="material_abb_olive_green">
-    <material name="">
-      <color rgba="${colour_abb_olive_green}"/>
-    </material>
-  </xacro:macro>
-  <xacro:macro name="material_abb_gray_white">
-    <material name="">
-      <color rgba="${colour_abb_gray_white}"/>
-    </material>
-  </xacro:macro>
-  <xacro:macro name="material_abb_pure_white">
-    <material name="">
-      <color rgba="${colour_abb_pure_white}"/>
-    </material>
-  </xacro:macro>
-  <xacro:macro name="material_abb_yellow">
-    <material name="">
-      <color rgba="${colour_abb_yellow}"/>
-    </material>
-  </xacro:macro>
+  <material name="abb_orange">
+    <color rgba="${colour_abb_orange}"/>
+  </material>
+  <material name="abb_graphite_white">
+    <color rgba="${colour_abb_graphite_white}"/>
+  </material>
+  <material name="abb_white">
+    <color rgba="${colour_abb_white}"/>
+  </material>
+  <material name="abb_pebble_gray">
+    <color rgba="${colour_abb_pebble_gray}"/>
+  </material>
+  <material name="abb_dark_gray">
+    <color rgba="${colour_abb_dark_gray}"/>
+  </material>
+  <material name="abb_black">
+    <color rgba="${colour_abb_black}"/>
+  </material>
+  <material name="abb_signal_red">
+    <color rgba="${colour_abb_signal_red}"/>
+  </material>
+  <material name="abb_carmine_red">
+    <color rgba="${colour_abb_carmine_red}"/>
+  </material>
+  <material name="abb_ultramarine_blue">
+    <color rgba="${colour_abb_ultramarine_blue}"/>
+  </material>
+  <material name="abb_sky_blue">
+    <color rgba="${colour_abb_sky_blue}"/>
+  </material>
+  <material name="abb_leaf_green">
+    <color rgba="${colour_abb_leaf_green}"/>
+  </material>
+  <material name="abb_olive_green">
+    <color rgba="${colour_abb_olive_green}"/>
+  </material>
+  <material name="abb_gray_white">
+    <color rgba="${colour_abb_gray_white}"/>
+  </material>
+  <material name="abb_pure_white">
+    <color rgba="${colour_abb_pure_white}"/>
+  </material>
+  <material name="abb_yellow">
+    <color rgba="${colour_abb_yellow}"/>
+  </material>
 </robot>

Commit message: heng

File: install/workcell_description/share/workcell_description/urdf/materials/common_materials.xacro (robot description, xacro)
@@ -2,5 +2,4 @@
 <robot xmlns:xacro="http://ros.org/wiki/xacro">
   <xacro:include filename="../materials/common_colours.xacro"/>
-  <!-- Global material definitions for reuse across links -->
   <material name="abb_orange">
     <color rgba="${colour_abb_orange}"/>

File: install/workcell_description/share/workcell_description/urdf/robots/irb6700_200_260.xacro (robot description, xacro)
@@ -1,6 +1,4 @@
 <?xml version="1.0"?>
 <robot xmlns:xacro="http://ros.org/wiki/xacro">
-  <!-- include common materials -->
-  <xacro:include filename="../materials/common_materials.xacro"/>
 <xacro:macro name="irb6700_link" params="prefix mesh_scale_visual:='1 1 1' mesh_scale_collision:='1 1 1' name mass ixx iyy izz">
   <link name="${prefix}${name}">

File: src/workcell_description/urdf/materials/common_materials.xacro (robot description, xacro)
@@ -47,3 +47,49 @@
     <color rgba="${colour_abb_yellow}"/>
   </material>
+  <!-- Convenience macros referencing the named materials -->
+  <xacro:macro name="material_abb_orange">
+    <material name="abb_orange"/>
+  </xacro:macro>
+  <xacro:macro name="material_abb_graphite_white">
+    <material name="abb_graphite_white"/>
+  </xacro:macro>
+  <xacro:macro name="material_abb_white">
+    <material name="abb_white"/>
+  </xacro:macro>
+  <xacro:macro name="material_abb_pebble_gray">
+    <material name="abb_pebble_gray"/>
+  </xacro:macro>
+  <xacro:macro name="material_abb_dark_gray">
+    <material name="abb_dark_gray"/>
+  </xacro:macro>
+  <xacro:macro name="material_abb_black">
+    <material name="abb_black"/>
+  </xacro:macro>
+  <xacro:macro name="material_abb_signal_red">
+    <material name="abb_signal_red"/>
+  </xacro:macro>
+  <xacro:macro name="material_abb_carmine_red">
+    <material name="abb_carmine_red"/>
+  </xacro:macro>
+  <xacro:macro name="material_abb_ultramarine_blue">
+    <material name="abb_ultramarine_blue"/>
+  </xacro:macro>
+  <xacro:macro name="material_abb_sky_blue">
+    <material name="abb_sky_blue"/>
+  </xacro:macro>
+  <xacro:macro name="material_abb_leaf_green">
+    <material name="abb_leaf_green"/>
+  </xacro:macro>
+  <xacro:macro name="material_abb_olive_green">
+    <material name="abb_olive_green"/>
+  </xacro:macro>
+  <xacro:macro name="material_abb_gray_white">
+    <material name="abb_gray_white"/>
+  </xacro:macro>
+  <xacro:macro name="material_abb_pure_white">
+    <material name="abb_pure_white"/>
+  </xacro:macro>
+  <xacro:macro name="material_abb_yellow">
+    <material name="abb_yellow"/>
+  </xacro:macro>
 </robot>
