Commit message: heng

File: install/workcell_description/share/workcell_description/urdf/robots/irb6700_200_260.xacro (robot description, xacro)
@@ -3,4 +3,27 @@
   <!-- include common materials -->
   <xacro:include filename="../materials/common_materials.xacro"/>
+<xacro:macro name="irb6700_link" params="prefix mesh_scale_visual:='1 1 1' mesh_scale_collision:='1 1 1' name mass ixx iyy izz">
+  <link name="${prefix}${name}">
+    <inertial>
+      <mass value="${mass}"/>
+      <origin xyz="0 0 0.1"/>
+      <inertia ixx="${ixx}" ixy="0" ixz="0" iyy="${iyy}" iyz="0" izz="${izz}"/>
+    </inertial>
+    <visual>
+      <origin xyz="0 0 0" rpy="0 0 0"/>
+      <geometry>
+        <mesh filename="package://workcell_description/meshes/robots/visual/${name}.stl" scale="${mesh_scale_visual}"/>
+      </geometry>
+      <xacro:material_abb_white/>
+    </visual>
+    <collision>
+      <origin xyz="0 0 0" rpy="0 0 0"/>
+      <geometry>
+        <mesh filename="package://workcell_description/meshes/robots/collision/${name}.stl" scale="${mesh_scale_collision}"/>
+      </geometry>
+      <xacro:material_abb_yellow/>
+    </collision>
+  </link>
+</xacro:macro>
 <xacro:macro name="irb6700_200_260"
              params="prefix mesh_scale_visual:='1 1 1' mesh_scale_collision:='1 1 1'">

File: install/workcell_description/share/workcell_description/urdf/workcell.urdf.xacro (robot description, xacro)
@@ -1,4 +1,4 @@
-<?xml version="1.0" encoding="UTF-8"?>
-<robot xmlns:xacro="http://www.ros.org/wiki/xacro" name="workcell">
+<?xml version="1.0"?>
+<robot xmlns:xacro="http://ros.org/wiki/xacro" name="workcell">
   <xacro:include filename="props/common_props.xacro"/>
   <xacro:include filename="materials/common_materials.xacro"/>

Commit message: can control robot

File: install/workcell_description/share/workcell_description/urdf/robots/irb6700_200_260.xacro (robot description, xacro)
@@ -13,5 +13,4 @@
         <mesh filename="package://workcell_description/meshes/robots/visual/${name}.stl" scale="${mesh_scale_visual}"/>
       </geometry>
-      <xacro:material_abb_white/>
     </visual>
     <collision>
@@ -20,5 +19,4 @@
         <mesh filename="package://workcell_description/meshes/robots/collision/${name}.stl" scale="${mesh_scale_collision}"/>
       </geometry>
-      <xacro:material_abb_yellow/>
     </collision>
   </link>
@@ -38,5 +36,4 @@
           <mesh filename="package://workcell_description/meshes/robots/visual/base_link.stl" scale="${mesh_scale_visual}"/>
         </geometry>
-        <xacro:material_abb_white/>
       </visual>
       <collision>
@@ -45,5 +42,4 @@
           <mesh filename="package://workcell_description/meshes/robots/collision/base_link.stl" scale="${mesh_scale_collision}"/>
         </geometry>
-        <xacro:material_abb_yellow/>
       </collision>
     </link>

File: install/workcell_description/share/workcell_description/urdf/workcell.urdf.xacro (robot description, xacro)
@@ -1,8 +1,18 @@
 <?xml version="1.0"?>
 <robot xmlns:xacro="http://ros.org/wiki/xacro" name="workcell">
-  <xacro:include filename="props/common_props.xacro"/>
-  <xacro:include filename="materials/common_materials.xacro"/>
-  <xacro:include filename="robots/irb6700_200_260.xacro"/>
-  <xacro:include filename="actuators/spindle.xacro"/>
+  <xacro:arg name="use_fake_hardware" default="true"/>
+  <xacro:property name="use_fake_hardware" value="$(arg use_fake_hardware)"/>
+  <xacro:arg name="rws_ip"            default="None"/>
+  <xacro:property name="rws_ip"            value="$(arg rws_ip)"/>
+  <xacro:arg name="rws_port"         default="80"/>
+  <xacro:property name="rws_port"         value="$(arg rws_port)"/>
+  <xacro:arg name="configure_via_rws" default="true"/>
+  <xacro:property name="configure_via_rws" value="$(arg configure_via_rws)"/>
+  <xacro:arg name="prefix" default=""/>
+  <xacro:arg name="mesh_scale_visual" default="1 1 1"/>
+  <xacro:arg name="mesh_scale_collision" default="1 1 1"/>
+  <xacro:include filename="$(find workcell_description)/urdf/props/common_props.xacro"/>
+  <xacro:include filename="$(find workcell_description)/urdf/robots/irb6700_200_260.xacro"/>
+  <xacro:include filename="$(find workcell_description)/urdf/actuators/spindle.xacro"/>
   <xacro:irb6700_200_260
       prefix="${prefix}"
@@ -15,3 +25,11 @@
       scale_v="${mesh_scale_visual}" scale_c="${mesh_scale_collision}"
       tcp_offset="0.150"/>
+  <xacro:include filename="$(find workcell_config)/config/workcell.ros2_control.xacro"/>
+  <xacro:workcell_ros2_control
+    name="ABBMultiInterfaceHardware"
+    use_fake_hardware="${use_fake_hardware}"
+    rws_ip="${rws_ip}"
+    rws_port="${rws_port}"
+    configure_via_rws="${configure_via_rws}"
+    initial_positions_file="$(find workcell_config)/config/initial_positions.yaml"/>
 </robot>
